Commit message: bug fix

File: robots/naviton.urdf.xacro (robot description, xacro)
@@ -6,4 +6,6 @@
   <xacro:include filename="$(find kcctsim)/urdf/sensors/gim30/gim30.urdf.xacro"/>
   <xacro:include filename="$(find kcctsim)/urdf/sensors/lrf/lrf.urdf.xacro"/>
+  <!--<xacro:include filename="$(find kcctsim)/urdf/sensors/imu/imu.urdf.xacro"/>
+-->
   <!-- =============== Link & Joint =============== -->
   <!-- Base -->
@@ -32,4 +34,8 @@
   	<origin xyz="0.07395931 0 0.24578237"/>
   </xacro:gim30_v0>-->
+<!--
+  <xacro:imu prefix="top" parent="base_link">
+	<origin xyz="0.0 0.0 0.0" rpy="0 0 0"/>
+  </xacro:imu>-->
   <!-- Front LRF -->
   <xacro:lrf_v0 prefix="front" parent="base_link">

Commit message: add velodyne, imu

File: robots/naviton.urdf.xacro (robot description, xacro)
@@ -6,4 +6,6 @@
   <xacro:include filename="$(find kcctsim)/urdf/sensors/gim30/gim30.urdf.xacro"/>
   <xacro:include filename="$(find kcctsim)/urdf/sensors/lrf/lrf.urdf.xacro"/>
+  <xacro:include filename="$(find velodyne_description)/urdf/HDL-32E.urdf.xacro"/>
+  <xacro:include filename="$(find kcctsim)/urdf/sensors/imu/imu.urdf.xacro" />
   <!-- =============== Link & Joint =============== -->
   <!-- Base -->
@@ -68,4 +70,6 @@
   <xacro:wheel_gazebo_v0 prefix="left"/>
   <!-- <xacro:wheel_gazebo_control_v0 rate="25"/> -->
+  <!--IMU-->
+  <xacro:imu_macro prefix="imu" parent="base_link" xyz="0 0 0"/>
   <!-- LRF -->
   <xacro:lrf_gazebo_v0 topic_name="scan1" prefix="front"
@@ -75,3 +79,7 @@
 					   min_rad="-2.35619449019" max_rad="1.65619449019"
 					   min_range="0.10" max_range="60.0"/>
+  <!-- VHDL-32E -->
+  <HDL-32E parent="base_link" name="velodyne" topic="velodyne_points" hz="10" samples="1024" gpu="false">
+      <origin xyz="0 0 0.8" rpy="0 0 0" />
+  </HDL-32E>
 </robot>

Commit message: base_foot_point 廃止

File: robots/naviton.urdf.xacro (robot description, xacro)
@@ -10,6 +10,6 @@
   <!-- =============== Link & Joint =============== -->
   <!-- Base -->
-  <link name="base_foot_point"/>
-  <xacro:base_v0 parent="base_foot_point">
+  <link name="base_link"/>
+  <xacro:base_v0 parent="base_link">
 	<origin xyz="0 0 0.0"/>
   </xacro:base_v0>

File: urdf/base/base.urdf.xacro (robot description, xacro)
@@ -6,7 +6,7 @@
 	  <insert_block name="joint_origin"/>
 	  <parent link="${parent}"/>
-	  <child link="base_link"/>
+	  <child link="body_link"/>
 	</joint>
-	<link name="base_link">
+	<link name="body_link">
 	  <visual>
 		<geometry>

Commit message: urdf update

File: robots/naviton.urdf.xacro (robot description, xacro)
@@ -36,15 +36,27 @@
   <!-- Front LRF -->
   <xacro:lrf_v0 prefix="front" parent="base_link">
-  	<origin xyz="0.225 -0.245 0.195"/>
+  	<origin xyz="0.225 0.0 0.195"/>
   </xacro:lrf_v0>
+  <link name="2d_blue"/>
+    <joint name="2d_blue_joint" type="fixed">
+    <parent link="front_lrf_link"/>
+    <child link="2d_blue"/>
+    <origin xyz="0 0 0"/>
+  </joint>
   <!-- Rear LRF -->
   <xacro:lrf_v0 prefix="rear" parent="base_link">
-  	<origin xyz="-0.485 0.245 0.195" rpy="0 0 -${M_PI}"/>
+  	<origin xyz="-0.485 0.0 0.195" rpy="0 0 -${M_PI}"/>
   </xacro:lrf_v0>
+  <link name="2d_orange"/>
+    <joint name="2d_orange_joint" type="fixed">
+    <parent link="rear_lrf_link"/>
+    <child link="2d_orange"/>
+    <origin xyz="0 0 0"/>
+  </joint>
   <link name="camera_link"/>
-  <joint name="lrf_link_joint" type="fixed">
-	<parent link="base_link"/>
-	<child link="camera_link"/>
-	<origin xyz="0 0 0.195"/>
+    <joint name="lrf_link_joint" type="fixed">
+    <parent link="base_link"/>
+    <child link="camera_link"/>
+    <origin xyz="0 0 0.195"/>
   </joint>
 <!--
@@ -77,5 +89,5 @@
 					   min_range="0.10" max_range="60.0"/>
   <xacro:lrf_gazebo_v0 topic_name="scan2" prefix="rear"
-					   min_rad="-2.35619449019" max_rad="1.65619449019"
+					   min_rad="-1.65806278939" max_rad="1.65619449019"
 					   min_range="0.10" max_range="60.0"/>
   <!-- VHDL-32E -->
