Commit message: apply noetic

File: urdf/base/base.urdf.xacro (robot description, xacro)
@@ -15,5 +15,5 @@
 		</geometry>
 		<material name="gray">
-    <color rgba="0.8 0.8 0.8 2.0"/>
+    <color rgba="0.8 0.8 0.8 1.0"/>
   </material>
 	  </visual>

File: urdf/sensors/lrf/lrf.urdf.xacro (robot description, xacro)
@@ -5,5 +5,5 @@
   <xacro:macro name="lrf_v0" params="prefix parent *joint_origin">
 	<joint name="${prefix}_lrf_joint" type="fixed">
-	  <insert_block name="joint_origin"/>
+	  <xacro:insert_block name="joint_origin"/>
 	  <parent link="${parent}"/>
 	  <child link="${prefix}_lrf_link"/>
@@ -22,5 +22,5 @@
 	  <inertial>
 		<origin xyz="0 0 -0.0164"/>
-		<box_inertial mass="0.4" height="0.07" width="0.07" depth="0.08"/>
+		<xacro:box_inertial mass="0.4" height="0.07" width="0.07" depth="0.08"/>
 	  </inertial>
 	</link>

File: urdf/wheel/wheel.urdf.xacro (robot description, xacro)
@@ -4,13 +4,13 @@
   <xacro:include filename="$(find kcctsim)/urdf/wheel/wheel.transmission.xacro"/>
   <xacro:include filename="$(find kcctsim)/urdf/wheel/wheel.gazebo.xacro"/>
-  <property name="wheel_radius" value="0.1575"/>
-  <property name="wheel_length" value="0.032"/>
-  <property name="wheel_mass" value="2.0"/>
+  <xacro:property name="wheel_radius" value="0.1575"/>
+  <xacro:property name="wheel_length" value="0.032"/>
+  <xacro:property name="wheel_mass" value="2.0"/>
   <xacro:macro name="wheel_v0" params="prefix parent *joint_origin *joint_axis">
 	<joint name="${prefix}_wheel_joint" type="continuous">
-	  <insert_block name="joint_origin"/>
+	  <xacro:insert_block name="joint_origin"/>
 	  <parent link="${parent}"/>
 	  <child link="${prefix}_wheel_link"/>
-	  <insert_block name="joint_axis"/>
+	  <xacro:insert_block name="joint_axis"/>
 	</joint>
 	<link name="${prefix}_wheel_link">
@@ -21,5 +21,5 @@
 		</geometry>
 		<material name="black">
-    		<color rgba="0.2 0.2 0.2 2.0"/>
+    		<color rgba="0.2 0.2 0.2 1.0"/>
   		</material>
 	  </visual>
@@ -32,5 +32,6 @@
 	  <inertial>
 		<origin xyz="0 -0.003 0" rpy="${-M_PI/2} 0 0"/>
-		<cylinder_inertial mass="${wheel_mass}"
+		<mass value="${wheel_mass}"/>
+		<xacro:cylinder_inertial mass="${wheel_mass}"
 						   radius="${wheel_radius}" length="${wheel_length}"/>
 	  </inertial>
